Commit message: change of workspace

File: husky_ur10_cam/urdf/combined.urdf (robot description, URDF)
Before this commit: robot husky_ur10, 26 links, 25 joints
Links:
- link ur10_base_link_inertia: geometry collision mesh filename=file:///home/farhan/husky_ws/install/husky_ur10_cam/share/h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; visual mesh filename=file:///home/farhan/husky_ws/install/husky_ur10_cam/share/h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
- link ur10_forearm_link: geometry collision mesh filename=file:///home/farhan/husky_ws/install/husky_ur10_cam/share/h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; visual mesh filename=file:///home/farhan/husky_ws/install/husky_ur10_cam/share/h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
- link ur10_shoulder_link: geometry collision mesh filename=file:///home/farhan/husky_ws/install/husky_ur10_cam/share/h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; visual mesh filename=file:///home/farhan/husky_ws/install/husky_ur10_cam/share/h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
- link ur10_upper_arm_link: geometry collision mesh filename=file:///home/farhan/husky_ws/install/husky_ur10_cam/share/h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; visual mesh filename=file:///home/farhan/husky_ws/install/husky_ur10_cam/share/h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
- link ur10_wrist_1_link: geometry collision mesh filename=file:///home/farhan/husky_ws/install/husky_ur10_cam/share/h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; visual mesh filename=file:///home/farhan/husky_ws/install/husky_ur10_cam/share/h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
- link ur10_wrist_2_link: geometry collision mesh filename=file:///home/farhan/husky_ws/install/husky_ur10_cam/share/h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; visual mesh filename=file:///home/farhan/husky_ws/install/husky_ur10_cam/share/h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
- link ur10_wrist_3_link: geometry collision mesh filename=file:///home/farhan/husky_ws/install/husky_ur10_cam/share/h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; visual mesh filename=file:///home/farhan/husky_ws/install/husky_ur10_cam/share/h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

Commit message: fix depth camera frame issue

File: husky_ur10_cam/urdf/combined.urdf (robot description, URDF)
Before this commit: robot husky_ur10, 26 links, 25 joints
Links:
- link camera: mass None -> 1.0; geometry collision box size=0.02 0.10 0.02; visual box size=0.02 0.10 0.02
Joints:
- joint camera_joint: origin xyz=0 0 0.01 rpy=0 -1.5707963267948966 1.5707963267948966 -> xyz=0 0 0.01 rpy=1.5707963267948966 -1.5707963267948966 0
- joint camera_optical_joint: origin xyz=0 0 0 rpy=0 0 0 -> xyz=0 0 0 rpy=-1.5707963267948966 0 -1.5707963267948966
- joint ur10_flange-tool0: origin xyz=0 0 0 rpy=1.5707963267948966 0 1.5707963267948966 -> xyz=0 0 0 rpy=0 0 0
- joint ur10_wrist_3-flange: origin xyz=0 0 0 rpy=0 -1.5707963267948966 -1.5707963267948966 -> xyz=0 0 0 rpy=0 0 0

Commit message: visualize fake voxels

File: husky_ur10_cam/urdf/combined.urdf (robot description, URDF)
Before this commit: robot husky_ur10, 26 links, 25 joints
Joints:
- joint velodyne2_mount_joint: origin xyz=-0.30 0 0.141 rpy=0 0 0 -> xyz=-0.32 0 0.141 rpy=0 0 0
- joint velodyne_mount_joint: origin xyz=0.30 0 0.141 rpy=0 0 0 -> xyz=0.32 0 0.141 rpy=0 0 0
