Commit message: sync push

File: husky_ur10_moveit_config/srdf/ur_macro.srdf.xacro (robot description, xacro)
@@ -15,21 +15,61 @@
     </group>
     <!--GROUP STATES - Purpose - Define a named state for a particular group, in terms of joint values. This is useful to define states like 'folded arms'-->
-    <group_state name="${prefix}home" group="${prefix}${name}_manipulator">
-      <joint name="${prefix}elbow_joint" value="0" />
-      <joint name="${prefix}shoulder_lift_joint" value="-1.5707" />
+    <group_state name="front_low" group="${prefix}${name}_manipulator">
+      <joint name="${prefix}elbow_joint" value="2.30" />
+      <joint name="${prefix}shoulder_lift_joint" value="-1.83" />
       <joint name="${prefix}shoulder_pan_joint" value="0" />
-      <joint name="${prefix}wrist_1_joint" value="0" />
-      <joint name="${prefix}wrist_2_joint" value="0" />
-      <joint name="${prefix}wrist_3_joint" value="0" />
+      <joint name="${prefix}wrist_1_joint" value="-3.58" />
+      <joint name="${prefix}wrist_2_joint" value="-1.57" />
+      <joint name="${prefix}wrist_3_joint" value="0.0" />
     </group_state>
-    <group_state name="${prefix}up" group="${prefix}${name}_manipulator">
-      <joint name="${prefix}elbow_joint" value="0" />
-      <joint name="${prefix}shoulder_lift_joint" value="-1.5707" />
-      <joint name="${prefix}shoulder_pan_joint" value="0" />
-      <joint name="${prefix}wrist_1_joint" value="-1.5707" />
-      <joint name="${prefix}wrist_2_joint" value="0" />
-      <joint name="${prefix}wrist_3_joint" value="0" />
+    <group_state name="right_low" group="${prefix}${name}_manipulator">
+      <joint name="${prefix}elbow_joint" value="2.50" />
+      <joint name="${prefix}shoulder_lift_joint" value="-2.23" />
+      <joint name="${prefix}shoulder_pan_joint" value="-1.57" />
+      <joint name="${prefix}wrist_1_joint" value="-3.42" />
+      <joint name="${prefix}wrist_2_joint" value="-1.57" />
+      <joint name="${prefix}wrist_3_joint" value="0.0" />
     </group_state>
-    <group_state name="${prefix}test_configuration" group="${prefix}${name}_manipulator">
+    <group_state name="rear_low" group="${prefix}${name}_manipulator">
+      <joint name="${prefix}elbow_joint" value="2.37" />
+      <joint name="${prefix}shoulder_lift_joint" value="-1.95" />
+      <joint name="${prefix}shoulder_pan_joint" value="-3.14" />
+      <joint name="${prefix}wrist_1_joint" value="-3.58" />
+      <joint name="${prefix}wrist_2_joint" value="-1.57" />
+      <joint name="${prefix}wrist_3_joint" value="0.0" />
+    </group_state>
+    <group_state name="left_low" group="${prefix}${name}_manipulator">
+      <joint name="${prefix}elbow_joint" value="2.46" />
+      <joint name="${prefix}shoulder_lift_joint" value="-2.13" />
+      <joint name="${prefix}shoulder_pan_joint" value="-4.71" />
+      <joint name="${prefix}wrist_1_joint" value="-3.49" />
+      <joint name="${prefix}wrist_2_joint" value="-1.57" />
+      <joint name="${prefix}wrist_3_joint" value="0.0" />
+    </group_state>
+        <group_state name="front_high" group="${prefix}${name}_manipulator">
+      <joint name="${prefix}elbow_joint" value="1.4" />
+      <joint name="${prefix}shoulder_lift_joint" value="-1.62" />
+      <joint name="${prefix}shoulder_pan_joint" value="1.54" />
+      <joint name="${prefix}wrist_1_joint" value="-1.2" />
+      <joint name="${prefix}wrist_2_joint" value="-1.6" />
+      <joint name="${prefix}wrist_3_joint" value="-0.11" />
+    </group_state>
+    <group_state name="right_high" group="${prefix}${name}_manipulator">
+      <joint name="${prefix}elbow_joint" value="1.4" />
+      <joint name="${prefix}shoulder_lift_joint" value="-1.62" />
+      <joint name="${prefix}shoulder_pan_joint" value="1.54" />
+      <joint name="${prefix}wrist_1_joint" value="-1.2" />
+      <joint name="${prefix}wrist_2_joint" value="-1.6" />
+      <joint name="${prefix}wrist_3_joint" value="-0.11" />
+    </group_state>
+    <group_state name="rear_high" group="${prefix}${name}_manipulator">
+      <joint name="${prefix}elbow_joint" value="1.4" />
+      <joint name="${prefix}shoulder_lift_joint" value="-1.62" />
+      <joint name="${prefix}shoulder_pan_joint" value="1.54" />
+      <joint name="${prefix}wrist_1_joint" value="-1.2" />
+      <joint name="${prefix}wrist_2_joint" value="-1.6" />
+      <joint name="${prefix}wrist_3_joint" value="-0.11" />
+    </group_state>
+    <group_state name="left_high" group="${prefix}${name}_manipulator">
       <joint name="${prefix}elbow_joint" value="1.4" />
       <joint name="${prefix}shoulder_lift_joint" value="-1.62" />
